File: 3tastsp_v5_resistorcooldrive_battcheck/3tastsp_v5_resistorcooldrive_battcheck.sch (EAGLE design)
At the start: 27 parts, among them X1 2516-

Commit message: Update PCBs, add IR option
Parts:
- LICKSIG, TRIALSIG: value BNC_VERTICAL -> BNC_RIGHT_ANGLE; device open-ephys:BNC_VERTICAL -> connectors:BNC_RIGHT_ANGLE
- R1, R2, R3, R4, R5, R6, R7, R8, R9: device SparkFun-Resistors:RESISTORPTH-1/2W -> SparkFun-Resistors:1KOHM-1/4W-1%(PTH)HORIZ-KIT
Connections:
- net D10: now also R9.1; no longer R5.1
- net D11: now also R8.1; no longer R6.1
- net D7: now also R6.1; no longer R8.1
- net GND: now also R5.1; no longer R1.1
- net N$12: now also R2.2; no longer R4.2
- net N$13: now also R4.1; no longer R9.1
- net N$15: now also R2.1; no longer R4.1
- net N$16: now also R1.1; no longer R2.1
- net N$18: now also R5.2; no longer R1.2
- net N$2: now also TRIALSIG.SIG; no longer LICKSIG.SIGNAL
- net N$29: now also R4.2; no longer R9.2
- net N$3: now also LICKSIG.SIG; no longer TRIALSIG.SIGNAL
- net N$4: now also R6.2; no longer R8.2
- net N$7: now also R8.2; no longer R6.2
- net N$8: now also R9.2; no longer R5.2
- net N$9: now also R1.2; no longer R2.2
Other:
- moved on the sheet: R1, R2, R4, R5, R6, R8, R9
