File: sptinterface_v5_battcheck/spt_interface_v5_withbattcheck.sch (EAGLE design)
At the start: 32 parts, among them X1 2516-

Commit message: Update PCBs, add IR option
Parts:
- removed FLR: (no value), pinhead:PINHD-1X1
- added FLR2: (no value), pinhead:PINHD-1X1
- added JP3, JP5: (no value), pinhead:PINHD-1X3
- added JP6: (no value), pinhead:PINHD-1X4
- added R10, R11, R12, R13: (no value), SparkFun-Resistors:1KOHM-1/4W-5%(PTH)HORIZ-KIT
- added VRSWITCH: TIP122, transistor-npn:TIP122
- R1, R2, R3, R4, R5, R6, R7, R8, R9: device SparkFun-Resistors:RESISTORPTH-1/2W -> SparkFun-Resistors:1KOHM-1/4W-5%(PTH)HORIZ-KIT
Connections:
- new net N$29: VREG_5V.IN, VRSWITCH.E
- new net N$32: R1.2, VRSWITCH.B
- new net N$33: D1.C, R11.1
- new net N$36: JP6.4, R13.2
- net GND: now also FLR2.1, JP3.2, JP5.2, JP6.2; no longer FLR.1
- net N$1: now also R3.1; no longer R9.1
- net N$11: now also R6.1, R7.2; no longer R3.1, R4.2
- net N$12: now also R8.1, R9.2; no longer R1.1, R2.2
- net N$13: now also R7.1; no longer R4.1
- net N$14: now also R9.1; no longer R2.1
- net N$17: now also R10.2, R11.2; no longer D1.C, R5.2
- net N$18: now also JP3.1, R2.1, X1-3.KL; no longer R6.2
- net N$19: now also JP5.1, JP6.1, R2.2; no longer R6.1, X1-3.KL
- net N$2: now also VRSWITCH.C; no longer VREG_5V.IN
- net N$27: now also R6.2; no longer R3.2
- net N$28: now also JP5.3, JP6.3, R12.2; no longer JP4.3
- net N$3: now also R4.2; no longer R7.2
- net N$34: now also R5.1; no longer R8.2
- net N$35: now also R3.2; no longer R9.2
- net N$4: now also R5.2; no longer R8.1
- net N$5: now also R8.2; no longer R1.2
- net N$6: now also R10.1; no longer R5.1
- net N$7: now also R4.1; no longer R7.1
- net N$8: now also JP3.3, JP4.3, R1.1, R12.1, R13.1
Other:
- moved on the sheet: BATT, R1, R2, R3, R4, R5, R6, R7, R8, R9, SHLD
